File: eagle/norns-shield.brd (EAGLE design)
At the start: 85.1 x 80 mm, 80 parts, among them J1 TRS-IN, J2 TRS-OUT, J3 ISP-ROW, Q1 ASFL-12.288mhz, SW1 PVA1, SW2 PVA1, SW3 PVA1, U1 CS4270, X1 RASPI_BOARD_B+#_E3

Commit message: case stl
Connections:
- removed net N$11: J1.2, R7.2
- new net N$7: J1.3, R7.2
- net N$12: now also J1.2; no longer J1.3
- net N$15: now also J2.3; no longer J2.2
- net N$16: now also J2.2; no longer J2.3
Routing:
- net N$7: track 0.00 -> 20.3 mm
- net N$15: track 6.58 -> 21.1 mm
- net N$12: track 12.9 -> 7.64 mm
- net N$11: track 4.84 -> 0.00 mm
- net N$16: track 14.0 -> 11.0 mm
Other:
- board text added: "norns/shield 200323 monome.org"
- board text removed: "norns/shield 191106 monome.org"
