File: eagle/norns-shield.sch (EAGLE design)
At the start: 80 parts, among them J1 TRS-IN, J2 TRS-OUT, J3 ISP-ROW, Q1 ASFL-12.288mhz, SW1 PVA1, SW2 PVA1, SW3 PVA1, U1 CS4270, X1 RASPI_BOARD_B+#_E3

Commit message: case stl
Connections:
- removed net N$11: J1.T, R7.2
- new net N$7: J1.R, R7.2
- net N$12: now also J1.T; no longer J1.R
- net N$15: now also J2.R; no longer J2.T
- net N$16: now also J2.T; no longer J2.R
Changed lines of the file:
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@@
-</segment>
-</net>
-<net name="N$11" class="0">
-<segment>
-<pinref part="J1" gate="J$1" pin="T"/>
-<pinref part="R7" gate="G$1" pin="2"/>
-<wire x1="99.06" y1="93.98" x2="106.68" y2="93.98" width="0.1524" layer="91"/>
 </segment>
 </net>
 <net name="N$12" class="0">
 <segment>
-<pinref part="J1" gate="J$1" pin="R"/>
-<wire x1="99.06" y1="91.44" x2="104.14" y2="91.44" width="0.1524" layer="91"/>
 <wire x1="104.14" y1="91.44" x2="104.14" y2="66.04" width="0.1524" layer="91"/>
 <pinref part="R9" gate="G$1" pin="2"/>
 <wire x1="104.14" y1="66.04" x2="106.68" y2="66.04" width="0.1524" layer="91"/>
+<pinref part="J1" gate="J$1" pin="T"/>
+<wire x1="104.14" y1="91.44" x2="99.06" y2="93.98" width="0.1524" layer="91"/>
 </segment>
 </net>
@@
 <wire x1="200.66" y1="106.68" x2="203.2" y2="106.68" width="0.1524" layer="91"/>
 <wire x1="203.2" y1="106.68" x2="203.2" y2="104.14" width="0.1524" layer="91"/>
-<pinref part="J2" gate="J$1" pin="T"/>
-<wire x1="203.2" y1="106.68" x2="226.06" y2="106.68" width="0.1524" layer="91"/>
+<pinref part="J2" gate="J$1" pin="R"/>
+<wire x1="226.06" y1="104.14" x2="220.98" y2="106.68" width="0.1524" layer="91"/>
+<wire x1="220.98" y1="106.68" x2="203.2" y2="106.68" width="0.1524" layer="91"/>
 <junction x="203.2" y="106.68"/>
 </segment>
@@
 <wire x1="200.66" y1="78.74" x2="203.2" y2="78.74" width="0.1524" layer="91"/>
 <wire x1="203.2" y1="78.74" x2="203.2" y2="76.2" width="0.1524" layer="91"/>
-<pinref part="J2" gate="J$1" pin="R"/>
-<wire x1="226.06" y1="104.14" x2="220.98" y2="104.14" width="0.1524" layer="91"/>
 <wire x1="220.98" y1="104.14" x2="220.98" y2="78.74" width="0.1524" layer="91"/>
 <wire x1="220.98" y1="78.74" x2="203.2" y2="78.74" width="0.1524" layer="91"/>
 <junction x="203.2" y="78.74"/>
+<pinref part="J2" gate="J$1" pin="T"/>
+<wire x1="220.98" y1="104.14" x2="226.06" y2="106.68" width="0.1524" layer="91"/>
 </segment>
 </net>
@@
 </segment>
 </net>
+<net name="N$7" class="0">
+<segment>
+<pinref part="J1" gate="J$1" pin="R"/>
+<pinref part="R7" gate="G$1" pin="2"/>
+<wire x1="99.06" y1="91.44" x2="106.68" y2="93.98" width="0.1524" layer="91"/>
+</segment>
+</net>
